File: Circuit/incubator_main_board.kicad_pcb (KiCad board)
At the start: 2 copper layers, 68.1 x 69.8 mm, 25 parts, among them J1 Conn_01x20, J2 Conn_01x20, U1 AZ1117-3.3

Commit message: added PCB pdfs
Parts:
- removed H3: MountingHole, MountingHole:MountingHole_4.3mm_M4_DIN965_Pad_TopBottom
Changed lines of the file:
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@@
     )
-  )
-  (footprint "MountingHole:MountingHole_4.3mm_M4_DIN965_Pad_TopBottom" (layer "F.Cu")
-    (at 4.025 4.025)
-    (descr "Mounting Hole 4.3mm, M4, DIN965")
-    (tags "mounting hole 4.3mm m4 din965")
-    (property "Sheetfile" "incubator_main_board.kicad_sch")
-    (property "Sheetname" "")
-    (property "ki_description" "Mounting Hole without connection")
-    (property "ki_keywords" "mounting hole")
-    (attr exclude_from_pos_files)
-    (fp_text reference "H3" (at 0 -4.75) (layer "F.SilkS")
-        (effects (font (size 1 1) (thickness 0.15)))
-    )
-    (fp_text value "MountingHole" (at 0 4.75) (layer "F.Fab")
-        (effects (font (size 1 1) (thickness 0.15)))
-    )
-    (fp_text user "${REFERENCE}" (at 0 0) (layer "F.Fab")
-        (effects (font (size 1 1) (thickness 0.15)))
-    )
-    (fp_circle (center 0 0) (end 3.75 0)
-      (stroke (width 0.15) (type solid)) (fill none) (layer "Cmts.User"))
-    (fp_circle (center 0 0) (end 4 0)
-      (stroke (width 0.05) (type solid)) (fill none) (layer "F.CrtYd"))
-    (pad "1" thru_hole circle (at 0 0) (size 4.7 4.7) (drill 4.3) (layers "*.Cu" "*.Mask"))
-    (pad "1" connect circle (at 0 0) (size 7.5 7.5) (layers "F.Cu" "F.Mask"))
-    (pad "1" connect circle (at 0 0) (size 7.5 7.5) (layers "B.Cu" "B.Mask"))
   )
   (footprint "Connector_JST:JST_EH_B2B-EH-A_1x02_P2.50mm_Vertical" (layer "F.Cu")

Commit message: finished HAL layer
Parts:
- added H3: MountingHole, MountingHole:MountingHole_4.3mm_M4_DIN965_Pad_TopBottom, F.Cu at (4.03, 4.03)
Connections:
- J1 pad 11: MQ135_Digital -> unconnected-(J1-Pin_11-Pad11)
- MQ135 pad 1: unconnected-(MQ135-Pin_1-Pad1) -> Net-(MQ135-Pin_1)
- MQ135 pad 2: Net-(MQ135-Pin_2) -> unconnected-(MQ135-Pin_2-Pad2)
- NTC3950 pad 1: NTC3950 -> GND
- NTC3950 pad 2: Net-(NTC3950-Pin_2) -> NTC3950
- R2 pad 2: Net-(MQ135-Pin_2) -> Net-(MQ135-Pin_1)
- R4 pad 2: Net-(NTC3950-Pin_2) -> NTC3950
Routing:
- net Net-(MQ135-Pin_2): track 10.5 -> 0.00 mm
- net NTC3950: track 7.87 -> 15.9 mm
- net Net-(MQ135-Pin_1): track 0.00 -> 5.20 mm
- net Net-(NTC3950-Pin_2): track 4.51 -> 0.00 mm
- net GND: track 305.1 -> 307.7 mm
- net MQ135_Digital: track 10.1 -> 7.69 mm
Changed lines of the file:
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@@
   (net 34 "MotionSensor")
   (net 35 "NTC3950")
-  (net 36 "Net-(NTC3950-Pin_2)")
+  (net 36 "unconnected-(J1-Pin_11-Pad11)")
   (net 37 "SDA")
   (net 38 "SCL")
@@
   (net 41 "unconnected-(J2-Pin_8-Pad8)")
   (net 42 "MQ135_Digital")
-  (net 43 "unconnected-(MQ135-Pin_1-Pad1)")
-  (net 44 "Net-(MQ135-Pin_2)")
+  (net 43 "Net-(MQ135-Pin_1)")
+  (net 44 "unconnected-(MQ135-Pin_2-Pad2)")
   (footprint "Capacitor_THT:CP_Radial_D10.0mm_P5.00mm" (layer "F.Cu")
     (at 170.7388 65.471626 -90)
@@
       (net 8 "Humidifier") (pinfunction "Pin_10") (pintype "passive"))
     (pad "11" thru_hole oval (at 0 25.4) (size 1.7 1.7) (drill 1) (layers "*.Cu" "*.Mask")
-      (net 42 "MQ135_Digital") (pinfunction "Pin_11") (pintype "passive"))
+      (net 36 "unconnected-(J1-Pin_11-Pad11)") (pinfunction "Pin_11") (pintype "passive"))
     (pad "12" thru_hole oval (at 0 27.94) (size 1.7 1.7) (drill 1) (layers "*.Cu" "*.Mask")
       (net 14 "unconnected-(J1-Pin_12-Pad12)") (pinfunction "Pin_12") (pintype "passive"))
@@
       (net 42 "MQ135_Digital") (pintype "passive"))
     (pad "2" thru_hole oval (at 7.62 0 180) (size 1.6 1.6) (drill 0.8) (layers "*.Cu" "*.Mask")
-      (net 44 "Net-(MQ135-Pin_2)") (pintype "passive"))
+      (net 43 "Net-(MQ135-Pin_1)") (pintype "passive"))
     (model "${KICAD6_3DMODEL_DIR}/Resistor_THT.3dshapes/R_Axial_DIN0207_L6.3mm_D2.5mm_P7.62mm_Horizontal.wrl"
       (offset (xyz 0 0 0))
@@
       (stroke (width 0.1) (type solid)) (layer "F.Fab"))
     (pad "1" thru_hole roundrect (at 0 0 180) (size 1.7 1.95) (drill 0.95) (layers "*.Cu" "*.Mask") (roundrect_rratio 0.147059)
-      (net 43 "unconnected-(MQ135-Pin_1-Pad1)") (pinfunction "Pin_1") (pintype "passive"))
+      (net 43 "Net-(MQ135-Pin_1)") (pinfunction "Pin_1") (pintype "passive"))
     (pad "2" thru_hole oval (at 2.5 0 180) (size 1.7 1.95) (drill 0.95) (layers "*.Cu" "*.Mask")
-      (net 44 "Net-(MQ135-Pin_2)") (pinfunction "Pin_2") (pintype "passive"))
+      (net 44 "unconnected-(MQ135-Pin_2-Pad2)") (pinfunction "Pin_2") (pintype "passive"))
     (pad "3" thru_hole oval (at 5 0 180) (size 1.7 1.95) (drill 0.95) (layers "*.Cu" "*.Mask")
       (net 4 "GND") (pinfunction "Pin_3") (pintype "passive"))
@@
       (stroke (width 0.1) (type solid)) (layer "F.Fab"))
     (pad "1" thru_hole roundrect (at 0 0) (size 1.7 2) (drill 1) (layers "*.Cu" "*.Mask") (roundrect_rratio 0.147059)
-      (net 35 "NTC3950") (pinfunction "Pin_1") (pintype "passive"))
+      (net 4 "GND") (pinfunction "Pin_1") (pintype "passive"))
     (pad "2" thru_hole oval (at 2.5 0) (size 1.7 2) (drill 1) (layers "*.Cu" "*.Mask")
-      (net 36 "Net-(NTC3950-Pin_2)") (pinfunction "Pin_2") (pintype "passive"))
+      (net 35 "NTC3950") (pinfunction "Pin_2") (pintype "passive"))
     (model "${KICAD6_3DMODEL_DIR}/Connector_JST.3dshapes/JST_EH_B2B-EH-A_1x02_P2.50mm_Vertical.wrl"
       (offset (xyz 0 0 0))
@@
       (rotate (xyz 0 0 0))
     )
+  )
+  (footprint "MountingHole:MountingHole_4.3mm_M4_DIN965_Pad_TopBottom" (layer "F.Cu")
+    (at 4.025 4.025)
+    (descr "Mounting Hole 4.3mm, M4, DIN965")
+    (tags "mounting hole 4.3mm m4 din965")
+    (property "Sheetfile" "incubator_main_board.kicad_sch")
+    (property "Sheetname" "")
+    (property "ki_description" "Mounting Hole without connection")
+    (property "ki_keywords" "mounting hole")
+    (attr exclude_from_pos_files)
+    (fp_text reference "H3" (at 0 -4.75) (layer "F.SilkS")
+        (effects (font (size 1 1) (thickness 0.15)))
+    )
+    (fp_text value "MountingHole" (at 0 4.75) (layer "F.Fab")
+        (effects (font (size 1 1) (thickness 0.15)))
+    )
+    (fp_text user "${REFERENCE}" (at 0 0) (layer "F.Fab")
+        (effects (font (size 1 1) (thickness 0.15)))
+    )
+    (fp_circle (center 0 0) (end 3.75 0)
+      (stroke (width 0.15) (type solid)) (fill none) (layer "Cmts.User"))
+    (fp_circle (center 0 0) (end 4 0)
+      (stroke (width 0.05) (type solid)) (fill none) (layer "F.CrtYd"))
+    (pad "1" thru_hole circle (at 0 0) (size 4.7 4.7) (drill 4.3) (layers "*.Cu" "*.Mask"))
+    (pad "1" connect circle (at 0 0) (size 7.5 7.5) (layers "F.Cu" "F.Mask"))
+    (pad "1" connect circle (at 0 0) (size 7.5 7.5) (layers "B.Cu" "B.Mask"))
   )
   (footprint "Connector_JST:JST_EH_B2B-EH-A_1x02_P2.50mm_Vertical" (layer "F.Cu")
@@
       (net 6 "+3.3V") (pintype "passive"))
     (pad "2" thru_hole oval (at 7.62 0 180) (size 1.6 1.6) (drill 0.8) (layers "*.Cu" "*.Mask")
-      (net 36 "Net-(NTC3950-Pin_2)") (pintype "passive"))
+      (net 35 "NTC3950") (pintype "passive"))
     (model "${KICAD6_3DMODEL_DIR}/Resistor_THT.3dshapes/R_Axial_DIN0207_L6.3mm_D2.5mm_P7.62mm_Horizontal.wrl"
       (offset (xyz 0 0 0))
@@
   (segment (start 136.7488 110.2043) (end 137.5556 111.0111) (width 0.8) (layer "F.Cu") (net 4))
   (segment (start 170.7388 70.471626) (end 174.34879 70.471626) (width 0.8) (layer "F.Cu") (net 4))
+  (segment (start 174.3348 85.7866) (end 175.3108 84.8106) (width 0.8) (layer "F.Cu") (net 4))
   (segment (start 136.7488 110.2043) (end 138.8688 108.0843) (width 0.8) (layer "F.Cu") (net 4))
   (segment (start 162.3575 110.9225) (end 162.3575 121.2247) (width 0.8) (layer "F.Cu") (net 4))
@@
   (segment (start 163.430754 70.593149) (end 155.6258 70.593149) (width 0.8) (layer "F.Cu") (net 4))
   (segment (start 162.3575 92.4375) (end 150 80.08) (width 0.8) (layer "F.Cu") (net 4))
+  (segment (start 174.3348 87.0204) (end 174.3348 85.7866) (width 0.8) (layer "F.Cu") (net 4))
   (segment (start 184.538 110.6678) (end 184.538 118.7342) (width 0.8) (layer "F.Cu") (net 4))
   (segment (start 174.34879 70.471626) (end 190.5254 86.648236) (width 0.8) (layer "F.Cu") (net 4))
@@
   (segment (start 184.2662 99.9012) (end 184.2662 101.6762) (width 0.8) (layer "F.Cu") (net 34))
   (segment (start 182.225 97.86) (end 184.2662 99.9012) (width 0.8) (layer "F.Cu") (net 34))
-  (segment (start 171.0196 87.0204) (end 174.3348 87.0204) (width 0.8) (layer "F.Cu") (net 35))
-  (segment (start 167.8 90.24) (end 171.0196 87.0204) (width 0.8) (layer "F.Cu") (net 35))
-  (segment (start 180.8734 87.0204) (end 181.2036 87.3506) (width 0.8) (layer "F.Cu") (net 36))
-  (segment (start 176.8348 87.0204) (end 180.8734 87.0204) (width 0.8) (layer "F.Cu") (net 36))
+  (segment (start 180.8734 87.0204) (end 181.2036 87.3506) (width 0.8) (layer "F.Cu") (net 35))
+  (segment (start 167.8 90.24) (end 175.4152 90.24) (width 0.8) (layer "F.Cu") (net 35))
+  (segment (start 175.4152 90.24) (end 176.8348 88.8204) (width 0.8) (layer "F.Cu") (net 35))
+  (segment (start 176.8348 88.8204) (end 176.8348 87.0204) (width 0.8) (layer "F.Cu") (net 35))
+  (segment (start 176.8348 87.0204) (end 180.8734 87.0204) (width 0.8) (layer "F.Cu") (net 35))
   (segment (start 172.0658 115.64) (end 177.038 110.6678) (width 0.8) (layer "F.Cu") (net 37))
   (segment (start 167.8 115.64) (end 172.0658 115.64) (width 0.8) (layer "F.Cu") (net 37))
@@
   (segment (start 146.9452 120.72) (end 145.5166 122.1486) (width 0.8) (layer "F.Cu") (net 40))
   (segment (start 150 120.72) (end 146.9452 120.72) (width 0.8) (layer "F.Cu") (net 40))
-  (segment (start 148.2914 100.4) (end 146.4888 102.2026) (width 0.8) (layer "F.Cu") (net 42))
-  (segment (start 146.4888 102.2026) (end 146.4888 105.0109) (width 0.8) (layer "F.Cu") (net 42))
-  (segment (start 150 100.4) (end 148.2914 100.4) (width 0.8) (layer "F.Cu") (net 42))
+  (segment (start 146.4888 100.6926) (end 146.2786 100.4824) (width 0.8) (layer "F.Cu") (net 42))
+  (segment (start 146.4888 105.0109) (end 146.4888 100.6926) (width 0.8) (layer "F.Cu") (net 42))
   (segment (start 146.4888 108.0843) (end 146.4888 105.0109) (width 0.8) (layer "F.Cu") (net 42))
-  (segment (start 136.4742 102.8446) (end 136.7025 102.8446) (width 0.8) (layer "F.Cu") (net 44))
-  (segment (start 134.4422 102.87) (end 136.4488 102.87) (width 0.8) (layer "F.Cu") (net 44))
-  (segment (start 131.9746 106.9667) (end 131.9746 105.3376) (width 0.8) (layer "F.Cu") (net 44))
-  (segment (start 136.7025 102.8446) (end 138.8688 105.0109) (width 0.8) (layer "F.Cu") (net 44))
-  (segment (start 131.9746 105.3376) (end 134.4422 102.87) (width 0.8) (layer "F.Cu") (net 44))
-  (segment (start 136.4488 102.87) (end 136.4742 102.8446) (width 0.8) (layer "F.Cu") (net 44))
+  (segment (start 136.4304 105.0109) (end 134.4746 106.9667) (width 0.8) (layer "F.Cu") (net 43))
+  (segment (start 138.8688 105.0109) (end 136.4304 105.0109) (width 0.8) (layer "F.Cu") (net 43))
 )
