File: Circuit/incubator_main_board.kicad_sch (KiCad schematic)
At the start: 19 parts, among them J1 Conn_01x20, J2 Conn_01x20, Q2 S8050, U1 AZ1117-3.3

Commit message: further development in all components
Parts:
- removed J1, J2: Conn_01x20, symbol Connector_Generic:Conn_01x20
- removed Power12v3: Conn_01x02_Socket, Connector_JST:JST_EH_B2B-EH-A_1x02_P2.50mm_Vertical, symbol Connector:Conn_01x02_Socket
- removed Q2: S8050, Package_TO_SOT_THT:TO-92_Inline, symbol Transistor_BJT:S8050
- removed R1, R2: 10k, Resistor_THT:R_Axial_DIN0207_L6.3mm_D2.5mm_P7.62mm_Horizontal, symbol Device:R
- added Humidifier: Conn_01x03_Socket, Connector_JST:JST_EH_B3B-EH-A_1x03_P2.50mm_Vertical, symbol Connector:Conn_01x03_Socket
- added J1, J2: Conn_01x19_Socket, symbol Connector:Conn_01x19_Socket
- Blue_UV_Light: renamed from OLED2; value Conn_01x04_Socket -> Relay_2CH
- PSU_Control: renamed from Blue_Light; value Conn_01x03_Socket -> Relay_1CH
- renumbered Power12v4 to Buzzer
Other:
- moved on the sheet: Buzzer

Commit message: finished PCB layout
Parts:
- removed J1, J2: Conn_01x19_Socket, symbol Connector:Conn_01x19_Socket
- removed Power12v: Conn_01x02_Socket, Connector_JST:JST_EH_B2B-EH-A_1x02_P2.50mm_Vertical, symbol Connector:Conn_01x02_Socket
- added Button1: DIP, Resistor_THT:R_Axial_DIN0207_L6.3mm_D2.5mm_P5.08mm_Vertical, symbol Device:R
- added C1: 330uf, Capacitor_THT:CP_Radial_D10.0mm_P5.00mm, symbol Device:C_Polarized
- added C2: 220uf, Capacitor_THT:CP_Radial_D8.0mm_P5.00mm, symbol Device:C_Polarized
- added H1, H2: MountingHole, MountingHole:MountingHole_4.3mm_M4_DIN965_Pad_TopBottom, symbol Mechanical:MountingHole
- added J1, J2: Conn_01x20, Connector_PinSocket_2.54mm:PinSocket_1x20_P2.54mm_Vertical, symbol Connector_Generic:Conn_01x20
- added R1: 200, Resistor_THT:R_Axial_DIN0207_L6.3mm_D2.5mm_P7.62mm_Horizontal, symbol Device:R
- added R2: 1k, Resistor_THT:R_Axial_DIN0207_L6.3mm_D2.5mm_P7.62mm_Horizontal, symbol Device:R
- added R3: 2k, Resistor_THT:R_Axial_DIN0207_L6.3mm_D2.5mm_P7.62mm_Horizontal, symbol Device:R
- added R4: 100k, Resistor_THT:R_Axial_DIN0207_L6.3mm_D2.5mm_P7.62mm_Horizontal, symbol Device:R
- Buzzer1: renamed from Buzzer; value Conn_01x02_Socket -> JST2P
- DH22: value Conn_01x03_Socket -> JST3P
- Humidifier1: renamed from Humidifier; value Conn_01x03_Socket -> JST_3P
- LimitSwitch1: renamed from LimitSwitch; value Conn_01x02_Socket -> JST2P
- MQ135: value Conn_01x04_Socket -> JST4P
- MotionSensor1: renamed from MotionSensor; value Conn_01x03_Socket -> JST3P
- OLED1: renamed from OLED; value Conn_01x04_Socket -> JST4P
- Power5v1: renamed from Power5v; value Conn_01x02_Socket -> JST2P
- renumbered Blue_UV_Light to Blue_UV1, PSU_Control to PSU1, PullUp to PullUp1
Connections:
- net +3.3V: now also DH22.2 (Pin_2), MotionSensor1.3 (Pin_3), OLED1.3 (Pin_3), PullUp1.1, U1.2 (VO), C2.1, J2.5 (Pin_5), R4.1
- net +5V: now also Blue_UV1.1 (Pin_1), Humidifier1.1 (Pin_1), MQ135.4 (Pin_4), PSU1.1 (Pin_1), Power5v1.2 (Pin_2), U1.3 (VI), C1.1
- net GND: now also Blue_UV1.4 (Pin_4), Buzzer1.2 (Pin_2), DH22.1 (Pin_1), Humidifier1.3 (Pin_3), MQ135.3 (Pin_3), MotionSensor1.1 (Pin_1), OLED1.4 (Pin_4), PSU1.3 (Pin_3), Power5v1.1 (Pin_1), U1.1 (GND), Button1.2, C1.2, C2.2, J1.3 (Pin_3), J2.13 (Pin_13), J2.3 (Pin_3), R3.1
- net SDA: now reaches OLED1.1 (Pin_1)
- net SDA: now also J2.17 (Pin_17)
- net SCL: now reaches OLED1.2 (Pin_2)
- net SCL: now also J2.16 (Pin_16)
- net BlueLight: now reaches Blue_UV1.2 (Pin_2)
- net BlueLight: now also J1.6 (Pin_6)
- net UVLight: now reaches Blue_UV1.3 (Pin_3)
- net UVLight: now also J1.5 (Pin_5)
- net Humidifier: now reaches Humidifier1.2 (Pin_2)
- net Humidifier: now also J1.10 (Pin_10)
- net DH22: now reaches DH22.3 (Pin_3)
- net DH22: now also J2.20 (Pin_20)
- net at PullUp1.2: now also LimitSwitch1.2 (Pin_2)
- net at MQ135.2 (Pin_2): now also R2.2
- net LimitSwitch: now reaches LimitSwitch1.1 (Pin_1)
- net LimitSwitch: now also J2.9 (Pin_9)
- net MotionSensor: now reaches MotionSensor1.2 (Pin_2)
- net MotionSensor: now also J2.10 (Pin_10)
- net NTC3950: now reaches NTC3950.1 (Pin_1)
- net NTC3950: now also J2.7 (Pin_7)
- net at NTC3950.2 (Pin_2): now also R4.2
- net at Buzzer1.1 (Pin_1): now also R1.2
- net MainPSU: now reaches PSU1.2 (Pin_2)
- net MainPSU: now also J1.2 (Pin_2)
- new net: Button1.1, J2.11 (Pin_11)
- new net Buzzer: J1.19 (Pin_19), R1.1
- new net MQ135_Digital: J1.11 (Pin_11), R2.1, R3.2
Other:
- note added: "Currents: ntc: 5/200k = 0.025mA limit_switch: 3.3/10k = 0.33mA dh22: 2.4mA mq135: 150mA relay*3: 200mA*3 buzzer: 20mA humidifier: 400mA OLED: 40mA MCU: 72mA total: 885.755mA"
- moved on the sheet: Blue_UV1, Buzzer1, DH22, Humidifier1, LimitSwitch1, MQ135, MotionSensor1, NTC3950, OLED1, PSU1, Power5v1, PullUp1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

Commit message: finished HAL layer
Connections:
- net GND: now also NTC3950.1 (Pin_1)
- net MQ135_Digital: no longer J1.11 (Pin_11)
- net NTC3950: now also NTC3950.2 (Pin_2), R4.2; no longer NTC3950.1 (Pin_1)
- net at MQ135.1 (Pin_1): now also R2.2
- net at MQ135.2 (Pin_2): no longer R2.2
Other:
- moved on the sheet: NTC3950, R2, R3
Changed lines of the file:
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@@
 (kicad_sch (version 20230121) (generator eeschema)
   (paper "A4")
-  (junction (at 85.09 124.46) (diameter 0) (color 0 0 0 0)
-  )
-  (wire (pts (xy 87.63 120.65) (xy 85.09 120.65))
+  (junction (at 85.09 127) (diameter 0) (color 0 0 0 0)
+  )
+  (wire (pts (xy 184.15 83.82) (xy 182.88 83.82))
     (stroke (width 0) (type default))
   )
-  (wire (pts (xy 85.09 120.65) (xy 85.09 124.46))
+  (wire (pts (xy 87.63 123.19) (xy 85.09 123.19))
+    (stroke (width 0) (type default))
+  )
+  (wire (pts (xy 184.15 81.28) (xy 182.88 81.28))
+    (stroke (width 0) (type default))
+  )
+  (wire (pts (xy 85.09 123.19) (xy 85.09 127))
     (stroke (width 0) (type default))
   )
@@
     (effects (font (size 1.27 1.27)) (justify left bottom))
   )
-  (global_label "MQ135_Digital" (shape input) (at 87.63 120.65 0) (fields_autoplaced)
+  (global_label "MQ135_Digital" (shape input) (at 87.63 123.19 0) (fields_autoplaced)
     (effects (font (size 1.27 1.27)) (justify left))
-    (property "Intersheetrefs" "${INTERSHEET_REFS}" (at 104.1617 120.65 0)
+    (property "Intersheetrefs" "${INTERSHEET_REFS}" (at 104.1617 123.19 0)
       (effects (font (size 1.27 1.27)) (justify left) hide)
     )
@@
     )
   )
-  (global_label "MQ135_Digital" (shape input) (at 114.3 107.95 180) (fields_autoplaced)
-    (effects (font (size 1.27 1.27)) (justify right))
-    (property "Intersheetrefs" "${INTERSHEET_REFS}" (at 97.7683 107.95 0)
-      (effects (font (size 1.27 1.27)) (justify right) hide)
-    )
-  )
-  (global_label "NTC3950" (shape input) (at 182.88 83.82 180) (fields_autoplaced)
-    (effects (font (size 1.27 1.27)) (justify right))
-    (property "Intersheetrefs" "${INTERSHEET_REFS}" (at 171.4887 83.82 0)
-      (effects (font (size 1.27 1.27)) (justify right) hide)
+  (global_label "MQ135_Digital" (shape input) (at 162.56 101.6 0) (fields_autoplaced)
+    (effects (font (size 1.27 1.27)) (justify left))
+    (property "Intersheetrefs" "${INTERSHEET_REFS}" (at 179.0917 101.6 0)
+      (effects (font (size 1.27 1.27)) (justify left) hide)
+    )
+  )
+  (global_label "NTC3950" (shape input) (at 182.88 81.28 90) (fields_autoplaced)
+    (effects (font (size 1.27 1.27)) (justify left))
+    (property "Intersheetrefs" "${INTERSHEET_REFS}" (at 182.88 69.8887 90)
+      (effects (font (size 1.27 1.27)) (justify left) hide)
     )
   )
@@
     )
   )
+  (symbol (lib_id "power:GND") (at 182.88 83.82 270) (unit 1)
+    (in_bom yes) (on_board yes) (dnp no) (fields_autoplaced)
+    (property "Reference" "#PWR032" (at 176.53 83.82 0)
+      (effects (font (size 1.27 1.27)) hide)
+    )
+    (property "Value" "GND" (at 179.07 83.82 90)
+      (effects (font (size 1.27 1.27)) (justify right))
+    )
+    (property "Footprint" "" (at 182.88 83.82 0)
+      (effects (font (size 1.27 1.27)) hide)
+    )
+    (property "Datasheet" "" (at 182.88 83.82 0)
+      (effects (font (size 1.27 1.27)) hide)
+    )
+    (pin "1")
+    (instances
+      (project "incubator_main_board"
+        (path "/fa09ba5b-9e92-4a20-ae99-cc63a276da9a"
+          (reference "#PWR032") (unit 1)
+        )
+      )
+    )
+  )
   (symbol (lib_id "Connector:Conn_01x04_Socket") (at 186.69 135.89 0) (unit 1)
     (in_bom yes) (on_board yes) (dnp no) (fields_autoplaced)
@@
     )
   )
-  (symbol (lib_id "power:GND") (at 92.71 124.46 90) (mirror x) (unit 1)
-    (in_bom yes) (on_board yes) (dnp no)
-    (property "Reference" "#PWR014" (at 99.06 124.46 0)
-      (effects (font (size 1.27 1.27)) hide)
-    )
-    (property "Value" "GND" (at 96.52 124.46 0)
-      (effects (font (size 1.27 1.27)))
-    )
-    (property "Footprint" "" (at 92.71 124.46 0)
-      (effects (font (size 1.27 1.27)) hide)
-    )
-    (property "Datasheet" "" (at 92.71 124.46 0)
+  (symbol (lib_id "power:GND") (at 92.71 127 90) (mirror x) (unit 1)
+    (in_bom yes) (on_board yes) (dnp no)
+    (property "Reference" "#PWR014" (at 99.06 127 0)
+      (effects (font (size 1.27 1.27)) hide)
+    )
+    (property "Value" "GND" (at 96.52 127 0)
+      (effects (font (size 1.27 1.27)))
+    )
+    (property "Footprint" "" (at 92.71 127 0)
+      (effects (font (size 1.27 1.27)) hide)
+    )
+    (property "Datasheet" "" (at 92.71 127 0)
       (effects (font (size 1.27 1.27)) hide)
     )
@@
     )
   )
-  (symbol (lib_id "Device:R") (at 81.28 124.46 270) (mirror x) (unit 1)
-    (in_bom yes) (on_board yes) (dnp no) (fields_autoplaced)
-    (property "Reference" "R2" (at 80.01 127 0)
-      (effects (font (size 1.27 1.27)) (justify right))
-    )
-    (property "Value" "1k" (at 82.55 127 0)
-      (effects (font (size 1.27 1.27)) (justify right))
-    )
-    (property "Footprint" "Resistor_THT:R_Axial_DIN0207_L6.3mm_D2.5mm_P7.62mm_Horizontal" (at 81.28 126.238 90)
-      (effects (font (size 1.27 1.27)) hide)
-    )
-    (property "Datasheet" "~" (at 81.28 124.46 0)
+  (symbol (lib_id "Device:R") (at 81.28 127 270) (mirror x) (unit 1)
+    (in_bom yes) (on_board yes) (dnp no) (fields_autoplaced)
+    (property "Reference" "R2" (at 80.01 129.54 0)
+      (effects (font (size 1.27 1.27)) (justify right))
+    )
+    (property "Value" "1k" (at 82.55 129.54 0)
+      (effects (font (size 1.27 1.27)) (justify right))
+    )
+    (property "Footprint" "Resistor_THT:R_Axial_DIN0207_L6.3mm_D2.5mm_P7.62mm_Horizontal" (at 81.28 128.778 90)
+      (effects (font (size 1.27 1.27)) hide)
+    )
+    (property "Datasheet" "~" (at 81.28 127 0)
       (effects (font (size 1.27 1.27)) hide)
     )
@@
     )
   )
-  (symbol (lib_id "Connector:Conn_01x02_Socket") (at 187.96 83.82 0) (mirror x) (unit 1)
-    (in_bom yes) (on_board yes) (dnp no) (fields_autoplaced)
-    (property "Reference" "NTC3950" (at 187.325 76.2 0)
-      (effects (font (size 1.27 1.27)))
-    )
-    (property "Value" "100k" (at 187.325 78.74 0)
-      (effects (font (size 1.27 1.27)))
-    )
-    (property "Footprint" "Connector_JST:JST_EH_B2B-EH-A_1x02_P2.50mm_Vertical" (at 187.96 83.82 0)
-      (effects (font (size 1.27 1.27)) hide)
-    )
-    (property "Datasheet" "~" (at 187.96 83.82 0)
+  (symbol (lib_id "Connector:Conn_01x02_Socket") (at 189.23 83.82 0) (mirror x) (unit 1)
+    (in_bom yes) (on_board yes) (dnp no) (fields_autoplaced)
+    (property "Reference" "NTC3950" (at 188.595 76.2 0)
+      (effects (font (size 1.27 1.27)))
+    )
+    (property "Value" "100k" (at 188.595 78.74 0)
+      (effects (font (size 1.27 1.27)))
+    )
+    (property "Footprint" "Connector_JST:JST_EH_B2B-EH-A_1x02_P2.50mm_Vertical" (at 189.23 83.82 0)
+      (effects (font (size 1.27 1.27)) hide)
+    )
+    (property "Datasheet" "~" (at 189.23 83.82 0)
       (effects (font (size 1.27 1.27)) hide)
     )
@@
     )
   )
-  (symbol (lib_id "Device:R") (at 88.9 124.46 270) (mirror x) (unit 1)
-    (in_bom yes) (on_board yes) (dnp no) (fields_autoplaced)
-    (property "Reference" "R3" (at 87.63 127 0)
-      (effects (font (size 1.27 1.27)) (justify right))
-    )
-    (property "Value" "2k" (at 90.17 127 0)
-      (effects (font (size 1.27 1.27)) (justify right))
-    )
-    (property "Footprint" "Resistor_THT:R_Axial_DIN0207_L6.3mm_D2.5mm_P7.62mm_Horizontal" (at 88.9 126.238 90)
-      (effects (font (size 1.27 1.27)) hide)
-    )
-    (property "Datasheet" "~" (at 88.9 124.46 0)
-      (effects (font (size 1.27 1.27)) hide)
-    )
+  (symbol (lib_id "Device:R") (at 88.9 127 270) (mirror x) (unit 1)
+    (in_bom yes) (on_board yes) (dnp no) (fields_autoplaced)
+    (property "Reference" "R3" (at 87.63 129.54 0)
+      (effects (font (size 1.27 1.27)) (justify right))
+    )
+    (property "Value" "2k" (at 90.17 129.54 0)
+      (effects (font (size 1.27 1.27)) (justify right))
+    )
+    (property "Footprint" "Resistor_THT:R_Axial_DIN0207_L6.3mm_D2.5mm_P7.62mm_Horizontal" (at 88.9 128.778 90)
+      (effects (font (size 1.27 1.27)) hide)
+    )
+    (property "Datasheet" "~" (at 88.9 127 0)
+      (effects (font (size 1.27 1.27)) hide)
+    )
